Commit message: gazebo_sim renamed

File: src/gazebo_sim/urdf/head.urdf (robot description, URDF)
Before this commit: robot head_model, 2 links, 1 joints
Links:
- link head_link: geometry collision box size=0.001 0.001 0.001; visual mesh filename=package://gazebo_sim/meshes/head.stl scale=0.0001 0.0001 0.0001

File: src/gazebo_sim/urdf/head_vrglass.urdf (robot description, URDF)
Before this commit: robot head_model, 2 links, 1 joints
Links:
- link head_link: geometry collision box size=0.12 0.12 0.12; visual mesh filename=package://gazebo_sim/meshes/head_model.stl scale=0.001 0.001 0.001

File: src/gazebo_sim/urdf/rviz_head.urdf (robot description, URDF)
Before this commit: robot myfirst, 2 links, 1 joints
Links:
- link head_link: geometry visual mesh filename=package://gazebo_sim/meshes/head.stl scale=0.0001 0.0001 0.0001

Commit message: head rotation corrected

File: src/gazebo_sim/urdf/head.urdf (robot description, URDF)
Before this commit: robot head_model, 2 links, 1 joints
Links:
- link head_link: geometry collision box size=0.001 0.001 0.001; visual mesh filename=/home/zulal/vr_pc_ws/src/gazebo_sim/meshes/head.stl scale=0.0001 0.0001 0.0001
